File: hw/baseline_project/baseline_project.kicad_sch (KiCad schematic)
At the start: 46 parts, among them IC1 LM4041CILPR, J1 AudioJack, J2 Header_4, SW1 RESET, SW101 UP, SW102 DOWN, SW103 LEFT, SW104 RIGHT, SW105 MODE, U1 TLV5616CP, U101 EK-TM4C123GXL, U102 ESP8266-01/ESP-01, U103 Adafruit ST7735R, U3 LM2937xMP, U4 MCP34119P

Commit message: before changing display
Parts:
- added H1, H2, H3, H4: ~, ECE445L:MountingHole_4_40, symbol ECE445L:MountingHole
- U103: footprint ECE445L:adafruit_st7735r -> ECE445L:adafruit_st7735r2
Connections:
- no-connect marks 14 -> 18
Changed lines of the file:
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@@
   (no_connect (at 60.96 41.91))
   (no_connect (at 60.96 74.93))
+  (no_connect (at 196.85 128.778))
+  (no_connect (at 197.104 133.096))
   (no_connect (at 60.96 36.83))
   (no_connect (at 60.96 62.23))
   (no_connect (at 60.96 69.85))
+  (no_connect (at 197.612 137.16))
   (no_connect (at 60.96 67.31))
   (no_connect (at 125.476 166.116))
+  (no_connect (at 197.358 123.952))
   (no_connect (at 60.96 52.07))
   (wire (pts (xy 125.73 30.48) (xy 135.89 30.48))
@@
         (path "/69b823fd-c065-40ff-9bb9-c5835555f3eb"
           (reference "#FLG0102") (unit 1)
+        )
+      )
+    )
+  )
+  (symbol (lib_id "ECE445L:MountingHole") (at 197.612 137.16 0) (unit 1)
+    (in_bom yes) (on_board yes) (dnp no) (fields_autoplaced)
+    (property "Reference" "H4" (at 193.802 135.128 0)
+      (effects (font (size 1.27 1.27)))
+    )
+    (property "Value" "~" (at 197.612 137.16 0)
+      (effects (font (size 1.27 1.27)))
+    )
+    (property "Footprint" "ECE445L:MountingHole_4_40" (at 197.612 137.16 0)
+      (effects (font (size 1.27 1.27)) hide)
+    )
+    (property "Datasheet" "" (at 197.612 137.16 0)
+      (effects (font (size 1.27 1.27)) hide)
+    )
+    (pin "1")
+    (instances
+      (project "baseline_project"
+        (path "/69b823fd-c065-40ff-9bb9-c5835555f3eb"
+          (reference "H4") (unit 1)
         )
       )
@@
       (effects (font (size 1.27 1.27)))
     )
-    (property "Footprint" "ECE445L:adafruit_st7735r" (at 110.49 74.93 0)
+    (property "Footprint" "ECE445L:adafruit_st7735r2" (at 110.49 74.93 0)
       (effects (font (size 1.27 1.27)) (justify bottom) hide)
     )
@@
     )
   )
+  (symbol (lib_id "ECE445L:MountingHole") (at 196.85 128.778 0) (unit 1)
+    (in_bom yes) (on_board yes) (dnp no) (fields_autoplaced)
+    (property "Reference" "H2" (at 193.04 126.746 0)
+      (effects (font (size 1.27 1.27)))
+    )
+    (property "Value" "~" (at 196.85 128.778 0)
+      (effects (font (size 1.27 1.27)))
+    )
+    (property "Footprint" "ECE445L:MountingHole_4_40" (at 196.85 128.778 0)
+      (effects (font (size 1.27 1.27)) hide)
+    )
+    (property "Datasheet" "" (at 196.85 128.778 0)
+      (effects (font (size 1.27 1.27)) hide)
+    )
+    (pin "1")
+    (instances
+      (project "baseline_project"
+        (path "/69b823fd-c065-40ff-9bb9-c5835555f3eb"
+          (reference "H2") (unit 1)
+        )
+      )
+    )
+  )
   (symbol (lib_id "ECE445L:HeadphoneJack") (at 143.002 155.194 0) (unit 1)
     (in_bom yes) (on_board yes) (dnp no) (fields_autoplaced)
@@
     )
   )
+  (symbol (lib_id "ECE445L:MountingHole") (at 197.358 123.952 0) (unit 1)
+    (in_bom yes) (on_board yes) (dnp no) (fields_autoplaced)
+    (property "Reference" "H1" (at 193.548 121.92 0)
+      (effects (font (size 1.27 1.27)))
+    )
+    (property "Value" "~" (at 197.358 123.952 0)
+      (effects (font (size 1.27 1.27)))
+    )
+    (property "Footprint" "ECE445L:MountingHole_4_40" (at 197.358 123.952 0)
+      (effects (font (size 1.27 1.27)) hide)
+    )
+    (property "Datasheet" "" (at 197.358 123.952 0)
+      (effects (font (size 1.27 1.27)) hide)
+    )
+    (pin "1")
+    (instances
+      (project "baseline_project"
+        (path "/69b823fd-c065-40ff-9bb9-c5835555f3eb"
+          (reference "H1") (unit 1)
+        )
+      )
+    )
+  )
   (symbol (lib_id "ECE445L:C") (at 46.736 120.142 0) (unit 1)
     (in_bom yes) (on_board yes) (dnp no)
@@
         )
       )
+    )
+  )
+  (symbol (lib_id "ECE445L:MountingHole") (at 197.104 133.096 0) (unit 1)
+    (in_bom yes) (on_board yes) (dnp no) (fields_autoplaced)
+    (property "Reference" "H3" (at 193.294 131.064 0)
+      (effects (font (size 1.27 1.27)))
+    )
+    (property "Value" "~" (at 197.104 133.096 0)
+      (effects (font (size 1.27 1.27)))
+    )
+    (property "Footprint" "ECE445L:MountingHole_4_40" (at 197.104 133.096 0)
+      (effects (font (size 1.27 1.27)) hide)
+    )
+    (property "Datasheet" "" (at 197.104 133.096 0)
+      (effects (font (size 1.27 1.27)) hide)
+    )
+    (pin "1")
+    (instances
+      (project "baseline_project"
+        (path "/69b823fd-c065-40ff-9bb9-c5835555f3eb"
+          (reference "H3") (unit 1)
+        )
+      )

Commit message: so far so good new display pcb
Parts:
- removed C102: 100nF, ECE445L:C_Axial_200mil, symbol Device:C_Small
- removed C104: 4.7uF, ECE445L:CP_Radial_Tantal200mil, symbol Device:C_Polarized_Small_US
- removed U103: Adafruit ST7735R, ECE445L:adafruit_st7735r2, symbol adafruit_st7735r:Adafruit ST7735R
- added C12: 100nF, ECE445L:C_Axial_200mil, symbol Device:C_Small
- added C13: 4.7uF, ECE445L:CP_Radial_Tantal200mil, symbol Device:C_Polarized_Small_US
- added U2: ILI_Display, ECE445L:TFT-320x240, symbol ILI9341:ILI_Display
Connections:
- net +3V3: now also C12.1, C13.1, U2.1 (VCC), U2.8 (LED)
- net GND: now also C12.2, C13.2, U2.2 (GND)
- net SDC_CS: now also U2.15 (SD_CS)
- net TFT_CS: now also U2.3 (CS)
- net TFT_D/C: now also U2.5 (DC)
- net TFT_MISO: now also U2.9 (MISO)
- net TFT_MOSI: now also U2.6 (MOSI)
- net TFT_RST: now also U2.4 (RST)
- net TFT_SCK: now also U2.7 (SCK)
- net Touch_CS: now reaches U101.J1_4 (PB1)
- net Touch_CS: now also U2.11 (T_CS)
- net SS2_SCLK: now reaches U101.J1_7 (PB4)
- net SS2_SCLK: now also U2.10 (T_CLK), U2.18 (SD_SCK)
- net Touch_IRQ: now reaches U101.J2_2 (PB2)
- net Touch_IRQ: now also U2.14 (T_IRQ)
- net SS2_TX: now reaches U101.J2_6 (PB7)
- net SS2_TX: now also U2.12 (T_DIN), U2.16 (SD_MOSI)
- net SS2_RX: now reaches U101.J2_7 (PB6)
- net SS2_RX: now also U2.13 (T_DO), U2.17 (SD_MISO)
- no-connect marks 18 -> 13
Other:
- note removed: "I2C0_SCK"
- note removed: "PWM0"
- note removed: "TACH"
