File: hw/baseline_project/ps33536_hjs2235_shp695_wtc534.kicad_pcb (KiCad board)
At the start: 2 copper layers, 93.5 x 153.7 mm, 50 parts, among them IC1 LM4041CILPR, J1 AudioJack, J2 Header_4, SW1 RESET, SW101 UP, SW102 DOWN, SW103 LEFT, SW104 RIGHT, SW105 MODE, U1 TLV5616CP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

Commit message: final pcb submission
Parts:
- removed JP1: Jumper_3_Open, ECE445L:PinHeader_1x03_P2.54mm_Vertical
- removed TP1: TP, ECE445L:Testpoint_1x02_P2.54mm
- moved R11 53.6 mm to (102.9, 140.7)
- moved H3 19.0 mm to (104.1, 25.2)
- moved H4 18.8 mm to (187.6, 25.2)
- moved H1 6.87 mm to (104.1, 168.9)
- moved H2 6.63 mm to (187.6, 168.9)
Connections:
- J1 pad R: /DAC_Amp_Ctrl -> /Amp_Out
- J1 pad S: GND -> Net-(J1-sleeve)
- J1 pad T: /DAC_Amp_Ctrl -> /Amp_Out
- R11 pad 1: /Amp_Out -> +3V3
- R11 pad 2: /Pot_Out -> /Volume_Ctrl
- U101 pad J1_2: unconnected-(U101-PB5-PadJ1_2) -> /Volume_Ctrl
- U4 pad 8: unconnected-(U4-VO2-Pad8) -> Net-(J1-sleeve)
Routing:
- net /Volume_Ctrl: track 0.00 -> 40.3 mm, vias 0 -> 1
- net Net-(J1-sleeve): track 0.00 -> 26.1 mm
- net /DAC_Amp_Ctrl: track 24.1 -> 0.00 mm
- net /Amp_Out: track 34.8 -> 50.7 mm
- net /Pot_Out: track 13.6 -> 0.00 mm
- net +3V3: track 227.3 -> 240.1 mm
- net GND: track 510.4 -> 505.6 mm
Other:
- board text added: "ECE445L Spring 2024 - TPod Prithvi Senthilkumar Joon Song Siddhant Pandit Wyatt Cole TA - Aeybel Varghese"
- board text removed: "DAC_Amp_Ctrl"
- board text removed: "ECE445L Final - TPod Prithvi Senthilkumar Joon Song Siddhant Pandit Wyatt Cole"
- board text removed: "Volume_Jmp"
