File: hw/baseline_project/ps33536_hjs2235_shp695_wtc534.kicad_sch (KiCad schematic)
At the start: 50 parts, among them IC1 LM4041CILPR, J1 AudioJack, J2 Header_4, SW1 RESET, SW101 UP, SW102 DOWN, SW103 LEFT, SW104 RIGHT, SW105 MODE, U1 TLV5616CP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

Commit message: pcb and lab 7 report done
Other:
- note added: "ECE445L Final - TPod Prithvi Senthilkumar Joon Song Siddhant Pandit Wyatt Cole"

Commit message: final pcb submission
Parts:
- removed JP1: Jumper_3_Open, ECE445L:PinHeader_1x03_P2.54mm_Vertical, symbol ECE445L:Jumper_3_Open
- removed TP1: TP, ECE445L:Testpoint_1x02_P2.54mm, symbol ECE445L:Testpoint
Connections:
- net DAC_Amp_Ctrl is gone; now on net Amp_Out: J1.R (ring), J1.T (tip)
- net Pot_Out is gone; now on net Volume_Ctrl: R11.2
- net +3V3: now also R11.1
- net Amp_Out: no longer R11.1
- net GND: no longer J1.S (sleeve)
- net Volume_Ctrl: now reaches U101.J1_2 (PB5)
- net at U4.8 (VO2): now also J1.S (sleeve)
- no-connect marks 13 -> 11
Other:
- moved on the sheet: R11
